File: WiFiShield.sch (EAGLE design)
At the start: 35 parts, among them IC1 MC74VHCT50A, IC2 74AHC1G125, IC4 SPX3819M5-L-3-3, IC5 CC3000MOD, J10 Test, J2 Mode, J8 ARDUINO-SHIELD_R3, J9 U.FL-R-SMT-1(10)

Commit message: Update schematic PDF
Other:
- note added: "Version 0.1"
- note removed: "Version 0.5"
Changed lines of the file:
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@@
 <wire x1="119.38" y1="175.26" x2="124.46" y2="175.26" width="0.1524" layer="93"/>
 <text x="147.32" y="12.7" size="3.048" layer="94">CC3000 Arduino-compatible WiFi Shield</text>
-<text x="147.32" y="6.858" size="1.778" layer="94">Version 0.5</text>
+<text x="147.32" y="6.858" size="1.778" layer="94">Version 0.1</text>
 <text x="169.926" y="9.398" size="1.778" layer="94">http://freetronics.com/wifishield</text>
 <frame x1="0" y1="0" x2="248.92" y2="185.42" columns="8" rows="5" layer="94"/>

Commit message: Swap R1 to be pulldown on enable
Connections:
- net !CC3000_CS_3V3: no longer R1.2
- net +3V3: no longer R1.1
- net CC3000_EN_5V: now also R1.1
- net GND: now also R1.2
Changed lines of the file:
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@@
 <attribute name="PACKAGE" value="0603"/>
 </part>
-<part name="U$25" library="freetronics-luke" deviceset="+3.3V" device="" value="+3V3"/>
 <part name="R1" library="freetronics-master-v1" deviceset="RESISTOR" device="0603" value="10k">
 <attribute name="PACKAGE" value="0603"/>
@@
 <part name="U$27" library="freetronics-master-v1.1" deviceset="USD-SOCKET" device="NEW"/>
 <part name="ANT1" library="freetronics-angus" deviceset="2500AT44M0400" device=""/>
+<part name="U$6" library="freetronics-luke" deviceset="GND" device=""/>
 </parts>
 <sheets>
@@
 <attribute name="PACKAGE" x="121.92" y="22.86" size="1.27" layer="96"/>
 </instance>
-<instance part="U$25" gate="G$1" x="27.94" y="99.06" smashed="yes" rot="MR0">
-<attribute name="VALUE" x="25.4" y="99.06" size="1.27" layer="96" rot="MR0"/>
-</instance>
 <instance part="R1" gate="G$1" x="27.94" y="88.9" smashed="yes" rot="R270">
 <attribute name="NAME" x="20.32" y="91.44" size="1.27" layer="95"/>
@@
 <attribute name="VALUE" x="220.98" y="58.42" size="1.27" layer="96" rot="MR0" align="bottom-right"/>
 </instance>
+<instance part="U$6" gate="G$1" x="27.94" y="78.74" rot="MR0"/>
 </instances>
 <busses>
@@
 <junction x="22.86" y="165.1"/>
 </segment>
+<segment>
+<pinref part="U$6" gate="G$1" pin="GND"/>
+<pinref part="R1" gate="G$1" pin="2"/>
+<wire x1="27.94" y1="81.28" x2="27.94" y2="83.82" width="0.1524" layer="91"/>
+</segment>
 </net>
 <net name="+3V3" class="0">
@@
 </segment>
 <segment>
-<pinref part="U$25" gate="G$1" pin="+3V3"/>
-<pinref part="R1" gate="G$1" pin="1"/>
-<wire x1="27.94" y1="93.98" x2="27.94" y2="96.52" width="0.1524" layer="91"/>
-</segment>
-<segment>
 <pinref part="U$26" gate="G$1" pin="+3V3"/>
 <pinref part="R2" gate="G$1" pin="1"/>
@@
 <wire x1="63.5" y1="40.64" x2="60.96" y2="40.64" width="0.1524" layer="91"/>
 <label x="78.74" y="53.594" size="1.27" layer="95"/>
-</segment>
-<segment>
-<pinref part="R1" gate="G$1" pin="2"/>
-<wire x1="27.94" y1="83.82" x2="27.94" y2="78.74" width="0.1524" layer="91"/>
-<wire x1="27.94" y1="78.74" x2="60.96" y2="78.74" width="0.1524" layer="91"/>
-<label x="43.18" y="78.994" size="1.27" layer="95"/>
 </segment>
 <segment>
@@
 <label x="22.86" y="15.494" size="1.27" layer="95"/>
 </segment>
-</net>
+<segment>
+<pinref part="R1" gate="G$1" pin="1"/>
+<wire x1="27.94" y1="93.98" x2="27.94" y2="96.52" width="0.1524" layer="91"/>
+<wire x1="27.94" y1="96.52" x2="12.7" y2="96.52" width="0.1524" layer="91"/>
+<label x="12.7" y="96.52" size="1.27" layer="95"/>
+</segment>
+</net>

Commit message: Swap SPX3819 LDO for AP2112K-3.3
Parts:
- removed C4: 10nF, freetronics-master-v1:CAP0603
- IC4: value SPX3819M5-L-3-3 -> AP2112K-3.3; device SparkFun:V_REG_LDOSMD -> freetronics-angus:V_REG_LDOSMD
- renumbered U$27 to SD1
Connections:
- removed net N$43: C4.2, IC4.BP
- net GND: no longer C4.1
Changed lines of the file:
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@@
 </part>
 <part name="U$61" library="freetronics-luke" deviceset="GND" device=""/>
-<part name="C4" library="freetronics-master-v1" deviceset="CAP" device="0603" value="10nF">
-<attribute name="PACKAGE" value="0603"/>
-</part>
 <part name="C5" library="freetronics-master-v1" deviceset="CAP" device="0603" value="1uF">
 <attribute name="PACKAGE" value="0603"/>
 </part>
-<part name="IC4" library="SparkFun" deviceset="V_REG_LDO" device="SMD" value="SPX3819M5-L-3-3">
+<part name="IC4" library="freetronics-angus" deviceset="V_REG_LDO" device="SMD" value="AP2112K-3.3">
 <attribute name="PACKAGE" value="5-SOT23"/>
 </part>
 <part name="U$15" library="freetronics-luke" deviceset="+3.3V" device="" value="+3V3"/>
-<part name="U$17" library="freetronics-luke" deviceset="GND" device=""/>
 <part name="U$18" library="freetronics-luke" deviceset="GND" device=""/>
 <part name="U$16" library="freetronics-luke" deviceset="GND" device=""/>
@@
 </part>
 <part name="U$10" library="freetronics-luke" deviceset="GND" device=""/>
-<part name="U$27" library="freetronics-master-v1.1" deviceset="USD-SOCKET" device="NEW"/>
+<part name="SD1" library="freetronics-master-v1.1" deviceset="USD-SOCKET" device="NEW"/>
 <part name="ANT1" library="freetronics-angus" deviceset="2500AT44M0400" device=""/>
 <part name="U$6" library="freetronics-luke" deviceset="GND" device=""/>
@@
 </instance>
 <instance part="U$61" gate="G$1" x="182.88" y="38.1" rot="MR0"/>
-<instance part="C4" gate="G$1" x="106.68" y="114.3" smashed="yes" rot="R180">
-<attribute name="NAME" x="99.06" y="111.76" size="1.27" layer="95"/>
-<attribute name="VALUE" x="99.06" y="109.22" size="1.27" layer="96"/>
-<attribute name="PACKAGE" x="99.06" y="106.68" size="1.27" layer="96"/>
-</instance>
 <instance part="C5" gate="G$1" x="119.38" y="111.76" smashed="yes">
 <attribute name="NAME" x="111.76" y="111.76" size="1.27" layer="95"/>
@@
 <attribute name="VALUE" x="111.76" y="134.62" size="1.27" layer="96"/>
 </instance>
-<instance part="U$17" gate="G$1" x="106.68" y="104.14" rot="MR0"/>
 <instance part="U$18" gate="G$1" x="119.38" y="104.14" rot="MR0"/>
 <instance part="U$16" gate="G$1" x="76.2" y="104.14" rot="MR0"/>
@@
 </instance>
 <instance part="U$10" gate="G$1" x="22.86" y="160.02" rot="MR0"/>
-<instance part="U$27" gate="G$1" x="22.86" y="129.54" rot="MR0"/>
+<instance part="SD1" gate="G$1" x="22.86" y="129.54" rot="MR0"/>
 <instance part="ANT1" gate="G$1" x="218.44" y="60.96" smashed="yes" rot="MR0">
 <attribute name="NAME" x="220.98" y="60.96" size="1.27" layer="95" rot="MR0" align="bottom-right"/>
@@
 </segment>
 <segment>
-<pinref part="C4" gate="G$1" pin="1"/>
-<wire x1="106.68" y1="106.68" x2="106.68" y2="109.22" width="0.1524" layer="91"/>
-<pinref part="U$17" gate="G$1" pin="GND"/>
-</segment>
-<segment>
 <pinref part="C5" gate="G$1" pin="2"/>
 <pinref part="U$18" gate="G$1" pin="GND"/>
@@
 <segment>
 <pinref part="U$2" gate="G$1" pin="GND"/>
-<pinref part="U$27" gate="G$1" pin="SHIELD1"/>
+<pinref part="SD1" gate="G$1" pin="SHIELD1"/>
 <wire x1="30.48" y1="114.3" x2="40.64" y2="114.3" width="0.1524" layer="91"/>
 <wire x1="40.64" y1="114.3" x2="40.64" y2="111.76" width="0.1524" layer="91"/>
-<pinref part="U$27" gate="G$1" pin="SHIELD2"/>
+<pinref part="SD1" gate="G$1" pin="SHIELD2"/>
 <wire x1="40.64" y1="111.76" x2="40.64" y2="106.68" width="0.1524" layer="91"/>
 <wire x1="30.48" y1="111.76" x2="40.64" y2="111.76" width="0.1524" layer="91"/>
 <junction x="40.64" y="111.76"/>
-<pinref part="U$27" gate="G$1" pin="GND"/>
+<pinref part="SD1" gate="G$1" pin="GND"/>
 <wire x1="30.48" y1="129.54" x2="40.64" y2="129.54" width="0.1524" layer="91"/>
 <wire x1="40.64" y1="129.54" x2="40.64" y2="114.3" width="0.1524" layer="91"/>
@@
 <pinref part="R4" gate="G$1" pin="2"/>
 <wire x1="50.8" y1="119.38" x2="48.26" y2="119.38" width="0.1524" layer="91"/>
-<pinref part="U$27" gate="G$1" pin="VCC"/>
+<pinref part="SD1" gate="G$1" pin="VCC"/>
 <wire x1="30.48" y1="134.62" x2="48.26" y2="134.62" width="0.1524" layer="91"/>
 <junction x="48.26" y="134.62"/>
@@
 </segment>
 </net>
-<net name="N$43" class="0">
-<segment>
-<wire x1="104.14" y1="119.38" x2="106.68" y2="119.38" width="0.1524" layer="91"/>
-<wire x1="106.68" y1="119.38" x2="106.68" y2="116.84" width="0.1524" layer="91"/>
-<pinref part="C4" gate="G$1" pin="2"/>
-<pinref part="IC4" gate="G$1" pin="BP"/>
-</segment>
-</net>
 <net name="N$28" class="0">
 <segment>
@@
 <wire x1="30.48" y1="132.08" x2="43.18" y2="132.08" width="0.1524" layer="91"/>
 <label x="33.02" y="132.334" size="1.27" layer="95"/>
-<pinref part="U$27" gate="G$1" pin="SCK"/>
+<pinref part="SD1" gate="G$1" pin="SCK"/>
 </segment>
 <segment>
@@
 <label x="33.02" y="137.414" size="1.27" layer="95"/>
 <wire x1="30.48" y1="137.16" x2="43.18" y2="137.16" width="0.1524" layer="91"/>
-<pinref part="U$27" gate="G$1" pin="DI"/>
+<pinref part="SD1" gate="G$1" pin="DI"/>
 </segment>
 <segment>
@@
 <pinref part="IC1" gate="A" pin="O"/>
 <label x="33.02" y="139.954" size="1.27" layer="95"/>
-<pinref part="U$27" gate="G$1" pin="CS"/>
+<pinref part="SD1" gate="G$1" pin="CS"/>
 <wire x1="30.48" y1="139.7" x2="55.88" y2="139.7" width="0.1524" layer="91"/>
 </segment>
@@
 </segment>
 <segment>
-<pinref part="U$27" gate="G$1" pin="DO"/>
+<pinref part="SD1" gate="G$1" pin="DO"/>
 <wire x1="30.48" y1="127" x2="38.1" y2="127" width="0.1016" layer="91"/>
 <label x="30.48" y="127" size="1.27" layer="95"/>
